File: pedals/Doctor Q/Doctor Q.kicad_sch (KiCad schematic)
At the start: 30 parts, among them J1 In, J2 Out, J3 +9v, Q1 2N3904, SW1 Norm/Bass, U1 RC4558

Commit message: Add files via upload
Parts:
- removed D1: 1N4148, Diode_THT:D_DO-35_SOD27_P7.62mm_Horizontal, symbol Diode:1N4148
- removed RV2: B25K, symbol Device:R_Potentiometer_Trim
- added C1: 50nF, symbol Device:C
- added C2: 10uF, symbol Device:C_Polarized
- added D3, D4: Red, symbol Device:LED
- added Q1: 2N5457, symbol Device:Q_NJFET_DSG
- added R13, R4: 10K, symbol Device:R
- added R2, R3: 1M, symbol Device:R
- added RV2: B25K, symbol Device:R_Potentiometer
- C3, C7: value 5nF -> 50nF
- renumbered Q1 to Q2, R6 to R1
Connections:
- net 9v: now also Q1.1 (D), R13.1, R2.1
- net GND: now also D3.1 (K), R3.2, R4.2, RV2.3; no longer U1.5 (+)
- net at D2.1 (K): now also RV2.1
- net at R11.2, U1.7: now also D4.2 (A)
- net Buffer: now reaches RV1.1, SW1.2 (B), SW1.6 (C)
- net Buffer: now also C2.2; no longer J1.1 (Pin_1)
- net at R12.1: now also D4.1 (K)
- net CV: now reaches R9.1
- net CV: now also RV2.2
- new net: C1.2, Q1.3 (G), R2.2, R3.1
- new net: D3.2 (A), R13.2, U1.5 (+)
- new net: C1.1, J1.1 (Pin_1)
- new net: C2.1, Q1.2 (S), R4.1
Other:
- note added: "Dr Quack Mod Add resistor and LED"
- note added: "Dr Quack Mod Potentiometer replaces trimpot"
- note added: "Dr Quack Mod Swap 1N914 for red LED"
- note added: "EHX Doctor Q Auto Wah with Mods"
- note added: "Envelope Follower"
- note added: "Input Buffer"
- note added: "MPF102 or other JFET as an alternative"
- note added: "Original had no input buffer"
- note added: "Originally ECG778 dual opamp TL072 would also be fine"
- note added: "Power"
- note added: "https://generalguitargadgets.com/effects-projects/filters-envelope/dr-quack-ehx-doctor-q/"
- note removed: "Originally ECG778 dual opamp"
- moved on the sheet: C1, C2, C3, C4, C5, C6, C7, C8, D2, J1, J2, Q2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
